File: M4_Video_Shield.kicad_pcb (KiCad board)
At the start: 2 copper layers, 68.6 x 53.3 mm, 20 parts, among them J1 Power, J2 Digital/PWM, J3 Analog, J4 Digital/PWM, J5 Video Out, U1 VS23S010D, Y1 4.433618MHz

Commit message: Route PCB
Parts:
- moved D1 13.4 mm to (125.4, 84.4)
- moved R3 12.9 mm to (120.0, 77.1)
- moved C2 12.5 mm to (148.3, 69.5), turned to -90 degrees
- moved R1 7.65 mm to (148.3, 71.7)
- moved Y1 6.33 mm to (153.3, 74.6)
- moved C5 6.03 mm to (138.1, 92.4)
- moved R2 5.80 mm to (125.7, 77.1)
- moved C1 5.25 mm to (148.3, 74.6), turned to 90 degrees
- moved C3 3.95 mm to (138.1, 87.3)
- moved C4 1.41 mm to (138.1, 81.8)
Routing:
- net /~{RESET}: track 0.00 -> 72.6 mm, vias 0 -> 2
- net /*11: track 0.00 -> 72.3 mm, vias 0 -> 1
- net /*9: track 0.00 -> 60.0 mm, vias 0 -> 1
- net /13: track 0.00 -> 54.0 mm, vias 0 -> 2
- net /*5: track 0.00 -> 49.4 mm
- net /PA23: track 0.00 -> 38.0 mm, vias 0 -> 2
- net +3V3: track 0.00 -> 37.0 mm
- net GND: track 0.00 -> 35.9 mm
- net /A0: track 0.00 -> 34.9 mm, vias 0 -> 2
- net /PA22: track 0.00 -> 33.7 mm, vias 0 -> 1
- net /4: track 0.00 -> 33.5 mm, vias 0 -> 2
- net /8: track 0.00 -> 28.5 mm, vias 0 -> 3
- net /A3: track 0.00 -> 28.1 mm
- net /A2: track 0.00 -> 27.2 mm
- net /*6: track 0.00 -> 26.9 mm
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- added copper zone on B.Cu, net GND
- added copper zone on F.Cu, net GND
