File: M4_Video_Shield.kicad_sch (KiCad schematic)
At the start: 16 parts, among them J1 Power, J2 Digital/PWM, J3 Analog, J4 Digital/PWM, J5 Video Out, U1 VS23S010D, Y1 4.433618MHz

Commit message: Route PCB
Parts:
- Y1: footprint (none) -> Crystal:Resonator-2Pin_W8.0mm_H3.5mm
Changed lines of the file:
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@@
       (effects (font (size 1.27 1.27)))
     )
-    (property "Footprint" "" (at 198.12 41.91 0)
+    (property "Footprint" "Crystal:Resonator-2Pin_W8.0mm_H3.5mm" (at 198.12 41.91 0)
       (effects (font (size 1.27 1.27)) hide)
     )
